File: FlightComputer_CPU_V1.kicad_pcb (KiCad board)
At the start: 4 copper layers, 31.8 x 31.8 mm, 32 parts, among them J1 Female Back Left, J2 Male Back Right, J3 Male Front Left, J4 Female Front Right, U1 STM32H503CBUx, U2 LD2981-3.3, U3 W25Q128JVP, Y2 Crystal_GND24_Small

Commit message: Finished V2 board layout
Parts:
- added TP1: TestPoint, TestPoint:TestPoint_Pad_D1.0mm, F.Cu at (113.0, 59.9)
- added TP2: TestPoint, TestPoint:TestPoint_Pad_D1.0mm, F.Cu at (115.0, 59.9)
- added TP3: TestPoint, TestPoint:TestPoint_Pad_D1.0mm, F.Cu at (113.0, 61.9)
- added TP4: TestPoint, TestPoint:TestPoint_Pad_D1.0mm, F.Cu at (115.0, 61.9)
- moved C20 0.25 mm to (99.7, 76.6)
- moved D4 0.22 mm to (99.9, 61.0)
- moved R40 0.22 mm to (103.8, 62.0)
- moved R41 0.22 mm to (103.8, 61.0)
- moved R42 0.22 mm to (103.8, 60.0)
Routing:
- net /I2C1_SCL: track 5.52 -> 35.0 mm, vias 2 -> 3
- net /I2C1_SDA: track 5.31 -> 30.5 mm, vias 1 -> 2
- net /SPI3_MISO: track 0.81 -> 23.2 mm, vias 1 -> 2
- net /IRQ_1: track 3.97 -> 26.0 mm, vias 1 -> 2
- net /IRQ_2: track 5.03 -> 24.6 mm, vias 2 -> 3
- net /I2C2_SDA: track 5.11 -> 23.0 mm, vias 1 -> 2
- net /USART1_RX: track 4.55 -> 21.8 mm
- net /SWDCLK: track 1.31 -> 18.3 mm, vias 1 -> 0
- net /LEDR: track 0.81 -> 16.8 mm, vias 1 -> 2
- net /FLASH_CS: track 2.27 -> 18.1 mm, vias 1 -> 2
- net /SPI3_SCK: track 0.81 -> 15.5 mm, vias 1 -> 2
- net /FDCAN1_RX: track 5.62 -> 19.4 mm
- net /LEDB: track 0.81 -> 13.0 mm, vias 1 -> 2
- net /USART2_RX: track 4.80 -> 16.6 mm
- net /SWDIO: track 1.06 -> 12.3 mm, vias 1 -> 0
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- added copper zone on F.Cu, net +5V
- added copper zone on In1.Cu, net +5V
- removed copper zone on In1.Cu, net +3V3_CPU
Other:
- board text added: "3V3"
- board text added: "GND"
- board text added: "SWD"
- board text added: "SWK"
