File: FlightComputer_CPU_V1.kicad_sch (KiCad schematic)
At the start: 71 parts, among them J1 Female Back Left, J2 Male Back Right, J3 Male Front Left, J4 Female Front Right, U1 STM32H503CBUx, U2 LD2981-3.3, U3 W25Q128JVP, Y2 Crystal_GND24_Small

Commit message: Finished V2 board layout
Other:
- moved on the sheet: C30, H1, H2, U3
